File: electronics/BaseESP8266.sch (KiCad schematic (older format))
At the start: 17 parts, among them P1 CONN_01X09, P2 CONN_01X09, SW1 Reset, T1 CONN_01X01, T2 CONN_01X01, U1 ESP-13-WROOM-02

Commit message: Most of BoM details added.  Part of #4
Parts:
- C2: Farnell (none) -> 2310565; Farnell Price/Stock (none) -> https://uk.farnell.com/multicomp/mc0603b473k250ct/cap-0-047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
- D4, D5, D6: Farnell (none) -> 2290332; Farnell Price/Stock (none) -> https://uk.farnell.com/kingbright/kp-2012seck/led-0805-250m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
- P1, P2, T1, T2: Description (none) -> DNP
- R1, R10, R2: Farnell (none) -> 2331740; Farnell Price/Stock (none) -> https://uk.farnell.com/te-connectivity/crgh0603j10k/res-10k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
- R6, R7, R8, R9: Farnell (none) -> 2502470; Farnell Price/Stock (none) -> https://uk.farnell.com/walsin/wr06x5600ftl/res-560r-1-75v-0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
- SW1: Farnell (none) -> 2435308; Farnell Price/Stock (none) -> http://uk.farnell.com/c-k-components/ksek43g-lfs/tactile-sw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
Changed lines of the file:
@@
 F 2 "Resistor_SMD:R_0603_1608Metric_Pad1.05x0.95mm_HandSolder" V 10230 3800 50  0001 C CNN
 F 3 "" H 10300 3800 50  0000 C CNN
+F 4 "2331740" V 10300 3800 50  0001 C CNN "Farnell"
+F 5 "https://uk.farnell.com/te-connectivity/crgh0603j10k/res-10k-5-0-2w-0603-thick-film/dp/2331740" V 10300 3800 50  0001 C CNN "Farnell Price/Stock"
 	1    10300 3800
 	-1   0    0    1
@@
 F 2 "TestPoint:TestPoint_Pad_D2.0mm" H 9800 2250 50  0001 C CNN
 F 3 "" H 9800 2250 50  0000 C CNN
+F 4 "DNP" H 9800 2250 50  0001 C CNN "Description"
 	1    9800 2250
 	1    0    0    -1
@@
 F 2 "TestPoint:TestPoint_Pad_D2.0mm" H 9600 3200 50  0001 C CNN
 F 3 "" H 9600 3200 50  0000 C CNN
+F 4 "DNP" V 9600 3200 50  0001 C CNN "Description"
 	1    9600 3200
 	0    1    1    0
@@
 F 2 "Capacitor_SMD:C_0603_1608Metric_Pad1.05x0.95mm_HandSolder" H 10788 3650 50  0001 C CNN
 F 3 "" H 10750 3800 50  0000 C CNN
+F 4 "2310565" V 10750 3800 50  0001 C CNN "Farnell"
+F 5 "https://uk.farnell.com/multicomp/mc0603b473k250ct/cap-0-047-f-25v-10-x7r-0603/dp/1759031" V 10750 3800 50  0001 C CNN "Farnell Price/Stock"
 	1    10750 3800
 	1    0    0    -1
@@
 F 2 "Resistor_SMD:R_0603_1608Metric_Pad1.05x0.95mm_HandSolder" V 5630 2000 50  0001 C CNN
 F 3 "" H 5700 2000 50  0000 C CNN
+F 4 "2502470" H 5700 2000 50  0001 C CNN "Farnell"
+F 5 "https://uk.farnell.com/walsin/wr06x5600ftl/res-560r-1-75v-0603-thick-film/dp/2502470" H 5700 2000 50  0001 C CNN "Farnell Price/Stock"
 	1    5700 2000
 	1    0    0    -1
@@
 F 2 "Resistor_SMD:R_0603_1608Metric_Pad1.05x0.95mm_HandSolder" V 9730 4000 50  0001 C CNN
 F 3 "" H 9800 4000 50  0000 C CNN
+F 4 "2502470" V 9800 4000 50  0001 C CNN "Farnell"
+F 5 "https://uk.farnell.com/walsin/wr06x5600ftl/res-560r-1-75v-0603-thick-film/dp/2502470" V 9800 4000 50  0001 C CNN "Farnell Price/Stock"
 	1    9800 4000
 	-1   0    0    1
@@
 F 2 "Resistor_SMD:R_0603_1608Metric_Pad1.05x0.95mm_HandSolder" V 9280 4000 50  0001 C CNN
 F 3 "" H 9350 4000 50  0000 C CNN
+F 4 "2502470" V 9350 4000 50  0001 C CNN "Farnell"
+F 5 "https://uk.farnell.com/walsin/wr06x5600ftl/res-560r-1-75v-0603-thick-film/dp/2502470" V 9350 4000 50  0001 C CNN "Farnell Price/Stock"
 	1    9350 4000
 	-1   0    0    1
@@
 F 2 "Resistor_SMD:R_0603_1608Metric_Pad1.05x0.95mm_HandSolder" V 8830 4000 50  0001 C CNN
 F 3 "" H 8900 4000 50  0000 C CNN
+F 4 "2502470" V 8900 4000 50  0001 C CNN "Farnell"
+F 5 "https://uk.farnell.com/walsin/wr06x5600ftl/res-560r-1-75v-0603-thick-film/dp/2502470" V 8900 4000 50  0001 C CNN "Farnell Price/Stock"
 	1    8900 4000
 	-1   0    0    1
@@
 F 2 "LED_SMD:LED_0805_2012Metric_Pad1.15x1.40mm_HandSolder" H 9800 3600 50  0001 C CNN
 F 3 "" H 9800 3600 50  0000 C CNN
+F 4 "2290332" H 9800 3600 50  0001 C CNN "Farnell"
+F 5 "https://uk.farnell.com/kingbright/kp-2012seck/led-0805-250mcd-orange/dp/2290332" H 9800 3600 50  0001 C CNN "Farnell Price/Stock"
 	1    9800 3600
 	0    -1   -1   0
@@
 F 2 "LED_SMD:LED_0805_2012Metric_Pad1.15x1.40mm_HandSolder" H 9350 3600 50  0001 C CNN
 F 3 "" H 9350 3600 50  0000 C CNN
+F 4 "2290332" H 9350 3600 50  0001 C CNN "Farnell"
+F 5 "https://uk.farnell.com/kingbright/kp-2012seck/led-0805-250mcd-orange/dp/2290332" H 9350 3600 50  0001 C CNN "Farnell Price/Stock"
 	1    9350 3600
 	0    -1   -1   0
@@
 F 2 "LED_SMD:LED_0805_2012Metric_Pad1.15x1.40mm_HandSolder" H 8900 3600 50  0001 C CNN
 F 3 "" H 8900 3600 50  0000 C CNN
+F 4 "2290332" H 8900 3600 50  0001 C CNN "Farnell"
+F 5 "https://uk.farnell.com/kingbright/kp-2012seck/led-0805-250mcd-orange/dp/2290332" H 8900 3600 50  0001 C CNN "Farnell Price/Stock"
 	1    8900 3600
 	0    -1   -1   0
@@
 F 2 "mcqn-kicad-lib:SW_SPST_GULLWING" H 9600 2650 50  0001 C CNN
 F 3 "" H 9600 2650 50  0000 C CNN
+F 4 "2435308" H 9600 2650 50  0001 C CNN "Farnell"
+F 5 "http://uk.farnell.com/c-k-components/ksek43g-lfs/tactile-switch-spst-0-05a-32vdc/dp/2435308" H 9600 2650 50  0001 C CNN "Farnell Price/Stock"
 	1    9600 2650
 	0    -1   -1   0
@@
 F 2 "Connector_PinSocket_2.54mm:PinSocket_1x09_P2.54mm_Vertical" H 1700 3250 50  0001 C CNN
 F 3 "" H 1700 3250 50  0000 C CNN
+F 4 "DNP" H 1700 3250 50  0001 C CNN "Description"
 	1    1700 3250
 	-1   0    0    1
@@
 F 2 "Connector_PinSocket_2.54mm:PinSocket_1x09_P2.54mm_Vertical" H 3650 3250 50  0001 C CNN
 F 3 "" H 3650 3250 50  0000 C CNN
+F 4 "DNP" H 3650 3250 50  0001 C CNN "Description"
 	1    3650 3250
 	1    0    0    -1
@@
 F 2 "Resistor_SMD:R_0603_1608Metric_Pad1.05x0.95mm_HandSolder" V 8430 4000 50  0000 C CNN
 F 3 "" H 8500 4000 50  0000 C CNN
+F 4 "2331740" V 8500 4000 50  0001 C CNN "Farnell"
+F 5 "https://uk.farnell.com/te-connectivity/crgh0603j10k/res-10k-5-0-2w-0603-thick-film/dp/2331740" V 8500 4000 50  0001 C CNN "Farnell Price/Stock"
 	1    8500 4000
 	-1   0    0    1
@@
 F 2 "Resistor_SMD:R_0603_1608Metric_Pad1.05x0.95mm_HandSolder" V 8480 2500 50  0000 C CNN
 F 3 "" H 8550 2500 50  0000 C CNN
+F 4 "2331740" H 8550 2500 50  0001 C CNN "Farnell"
+F 5 "https://uk.farnell.com/te-connectivity/crgh0603j10k/res-10k-5-0-2w-0603-thick-film/dp/2331740" H 8550 2500 50  0001 C CNN "Farnell Price/Stock"
 	1    8550 2500
 	1    0    0    -1

Commit message: Update one of the caps to cut-tape part rather than full reel.  Other minor tweaks.
Parts:
- C2: Farnell 2310565 -> 1759031
Changed lines of the file:
@@
 F 2 "Capacitor_SMD:C_0603_1608Metric_Pad1.05x0.95mm_HandSolder" H 10788 3650 50  0001 C CNN
 F 3 "" H 10750 3800 50  0000 C CNN
-F 4 "2310565" V 10750 3800 50  0001 C CNN "Farnell"
+F 4 "1759031" V 10750 3800 50  0001 C CNN "Farnell"
 F 5 "https://uk.farnell.com/multicomp/mc0603b473k250ct/cap-0-047-f-25v-10-x7r-0603/dp/1759031" V 10750 3800 50  0001 C CNN "Farnell Price/Stock"
 	1    10750 3800
